Commit message: feat: add inspectable gauge world assets

File: src/siminspect_description/urdf/siminspect.gazebo.xacro (robot description, xacro)
@@ -106,5 +106,5 @@
       <topic>/camera/image_raw</topic>
       <camera>
-        <horizontal_fov>1.0472</horizontal_fov>
+        <horizontal_fov>2.0</horizontal_fov>
         <image>
           <width>640</width>

File: src/siminspect_description/urdf/siminspect.urdf.xacro (robot description, xacro)
@@ -137,5 +137,5 @@
   </link>
   <joint name="camera_joint" type="fixed">
-    <origin xyz="0.18 0 0.12" rpy="0 0 0"/>
+    <origin xyz="0.18 0 0.70" rpy="0 0 0"/>
     <parent link="base_link"/>
     <child link="camera_link"/>
