Commit message: fix: align rolling geometry and bridge the IMU frame

File: src/siminspect_description/urdf/siminspect.urdf.xacro (robot description, xacro)
@@ -11,5 +11,5 @@
     <link name="${name}">
       <visual>
-        <origin xyz="0 0 0" rpy="0 0 0"/>
+        <origin xyz="0 0 0" rpy="${pi/2} 0 0"/>
         <geometry>
           <cylinder radius="0.075" length="0.04"/>
@@ -18,5 +18,5 @@
       </visual>
       <collision>
-        <origin xyz="0 0 0" rpy="0 0 0"/>
+        <origin xyz="0 0 0" rpy="${pi/2} 0 0"/>
         <geometry>
           <cylinder radius="0.075" length="0.04"/>
@@ -55,8 +55,13 @@
     </link>
     <joint name="${name}_joint" type="fixed">
-      <origin xyz="${x} ${y} -0.065" rpy="0 0 0"/>
+      <origin xyz="${x} ${y} -0.0825" rpy="0 0 0"/>
       <parent link="base_link"/>
       <child link="${name}"/>
     </joint>
+    <!-- A spherical caster approximates a freely swivelling support. -->
+    <gazebo reference="${name}">
+      <mu1>0.001</mu1>
+      <mu2>0.001</mu2>
+    </gazebo>
   </xacro:macro>
   <!-- ===== BASE LINK ===== -->
